Commit message: upload .usda file for the robot

File: robot_description/SO-ARM101-OMNI-KIN/Gripper.urdf (robot description, URDF)
Before this commit: robot Gripper, 4 links, 3 joints
Links:
- link base: geometry collision mesh filename=meshes/gripper_base.stl scale=0.001 0.001 0.001; visual mesh filename=meshes/gripper_base.stl scale=0.001 0.001 0.001
